Commit message: Update racecar.xacro

File: racecar.xacro (robot description, xacro)
@@ -37,18 +37,4 @@
       </geometry>
       <material name="black"/>
-    </visual>
-  </link>
-  <joint name="base_to_back_left_wheel" type="fixed">
-    <parent link="base_link"/>
-    <child link="back_left_wheel"/>
-    <origin xyz="0 ${(wheel_length+width)/2} ${wheel_radius}"/>
-  </joint>
-  <link name="back_left_wheel">
-    <visual>
-      <geometry>
-        <cylinder radius="${wheel_radius}" length="${wheel_length}"/>
-      </geometry>
-      <material name="black"/>
-      <origin rpy="${pi/2} 0 0"/>
     </visual>
   </link>

Commit message: Update racecar.xacro

File: racecar.xacro (robot description, xacro)
@@ -37,4 +37,18 @@
       </geometry>
       <material name="black"/>
+    </visual>
+  </link>
+ <joint name="base_to_back_left_wheel" type="fixed">
+    <parent link="base_link"/>
+    <child link="back_left_wheel"/>
+    <origin xyz="0 ${(wheel_length+width)/2} ${wheel_radius}"/>
+  </joint>
+  <link name="back_left_wheel">
+    <visual>
+      <geometry>
+        <cylinder radius="${wheel_radius}" length="${wheel_length}"/>
+      </geometry>
+      <material name="black"/>
+      <origin rpy="${pi/2} 0 0"/>
     </visual>
   </link>

Commit message: Update racecar.xacro

File: racecar.xacro (robot description, xacro)
@@ -40,16 +40,6 @@
   </link>
  <joint name="base_to_back_left_wheel" type="fixed">
-    <parent link="base_link"/>
-    <child link="back_left_wheel"/>
-    <origin xyz="0 ${(wheel_length+width)/2} ${wheel_radius}"/>
   </joint>
   <link name="back_left_wheel">
-    <visual>
-      <geometry>
-        <cylinder radius="${wheel_radius}" length="${wheel_length}"/>
-      </geometry>
-      <material name="black"/>
-      <origin rpy="${pi/2} 0 0"/>
-    </visual>
   </link>
   <joint name="base_to_back_right_wheel" type="fixed">

Commit message: Update racecar.xacro

File: racecar.xacro (robot description, xacro)
@@ -40,6 +40,16 @@
   </link>
  <joint name="base_to_back_left_wheel" type="fixed">
+    <parent link="base_link"/>
+    <child link="back_left_wheel"/>
+    <origin xyz="0 ${(wheel_length+width)/2} ${wheel_radius}"/>
   </joint>
   <link name="back_left_wheel">
+    <visual>
+      <geometry>
+        <cylinder radius="${wheel_radius}" length="${wheel_length}"/>
+      </geometry>
+      <material name="black"/>
+      <origin rpy="${pi/2} 0 0"/>
+    </visual>
   </link>
   <joint name="base_to_back_right_wheel" type="fixed">
